File: USB_adapter_v2.kicad_sch (KiCad schematic)
At the start: 24 parts, among them IC1 AP2112M-3.3TRG1, J1 10033527-N3112MLF, J2 Conn_02x10_Odd_Even, J3 Conn_01x05, J4 Standard?, Q1 BC847BDW1, SW1 SW_SPST, U1 CP2102NP1174GM, U2 D1213A-02SM

Commit message: f
Parts:
- removed SW1: SW_SPST, symbol Switch:SW_SPST
- added SW1: PTS526_SK15_SMTR2_LFS, PTS526SK15SMTR2LFS, symbol SamacSys_Parts:PTS526_SK15_SMTR2_LFS
Connections:
- net GND: now also SW1.3 (NO_1), SW1.4 (NO_2)
- net SW1: now reaches C1.1, R3.1, U1.9 (~{RST})
- net SW1: now also SW1.1 (COM_1), SW1.2 (COM_2)
Changed lines of the file:
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@@
+    (stroke (width 0) (type default) (color 0 0 0 0))
+  )
+  (wire (pts (xy 106.045 81.915) (xy 107.95 81.915))
     (stroke (width 0) (type default) (color 0 0 0 0))
   )
@@
     (stroke (width 0) (type default) (color 0 0 0 0))
   )
+  (wire (pts (xy 73.025 84.455) (xy 75.565 84.455))
+    (stroke (width 0) (type default) (color 0 0 0 0))
+  )
   (wire (pts (xy 221.615 48.26) (xy 221.615 38.1))
     (stroke (width 0) (type default) (color 0 0 0 0))
@@
     (stroke (width 0) (type default) (color 0 0 0 0))
   )
-  (wire (pts (xy 123.825 52.705) (xy 123.825 50.8))
-    (stroke (width 0) (type default) (color 0 0 0 0))
-  )
   (wire (pts (xy 167.005 57.785) (xy 156.845 57.785))
     (stroke (width 0) (type default) (color 0 0 0 0))
@@
     (stroke (width 0) (type default) (color 0 0 0 0))
   )
-  (wire (pts (xy 120.015 52.705) (xy 123.825 52.705))
+  (wire (pts (xy 73.025 81.915) (xy 75.565 81.915))
     (stroke (width 0) (type default) (color 0 0 0 0))
   )
@@
     (stroke (width 0) (type default) (color 0 0 0 0))
   )
+  (wire (pts (xy 106.045 84.455) (xy 107.95 84.455))
+    (stroke (width 0) (type default) (color 0 0 0 0))
+  )
   (wire (pts (xy 184.785 75.565) (xy 190.5 75.565))
     (stroke (width 0) (type default) (color 0 0 0 0))
@@
     (stroke (width 0) (type default) (color 0 0 0 0))
   )
-  (wire (pts (xy 123.825 50.8) (xy 127 50.8))
+  (wire (pts (xy 120.015 50.8) (xy 127 50.8))
     (stroke (width 0) (type default) (color 0 0 0 0))
   )
@@
     (effects (font (size 1.27 1.27)) (justify right bottom))
   )
+  (label "SW2" (at 73.025 84.455 180)
+    (effects (font (size 1.27 1.27)) (justify right bottom))
+  )
   (label "RI" (at 167.005 60.325 180)
     (effects (font (size 1.27 1.27)) (justify right bottom))
   )
+  (label "SW2" (at 120.015 50.8 0)
+    (effects (font (size 1.27 1.27)) (justify left bottom))
+  )
   (label "CTS" (at 167.005 50.165 180)
     (effects (font (size 1.27 1.27)) (justify right bottom))
   )
+  (label "SW2" (at 107.95 84.455 0)
+    (effects (font (size 1.27 1.27)) (justify left bottom))
+  )
+  (label "SW1" (at 73.025 81.915 180)
+    (effects (font (size 1.27 1.27)) (justify right bottom))
+  )
   (label "DTR" (at 109.22 147.955 0)
     (effects (font (size 1.27 1.27)) (justify left bottom))
@@
     (effects (font (size 1.27 1.27)) (justify right bottom))
   )
+  (label "SW1" (at 120.015 42.545 0)
+    (effects (font (size 1.27 1.27)) (justify left bottom))
+  )
   (label "GND" (at 248.285 133.35 180)
     (effects (font (size 1.27 1.27)) (justify right bottom))
@@
   (label "SUSPEND" (at 167.005 65.405 180)
     (effects (font (size 1.27 1.27)) (justify right bottom))
+  )
+  (label "SW1" (at 107.95 81.915 0)
+    (effects (font (size 1.27 1.27)) (justify left bottom))
   )
   (label "RXD" (at 167.005 45.085 180)
@@
     )
     (property "Datasheet" "~" (id 3) (at 226.06 48.26 0)
-      (effects (font (size 1.27 1.27)) hide)
-    )
-    (pin "1")
-    (pin "2")
-  )
-  (symbol (lib_id "Switch:SW_SPST") (at 120.015 47.625 90) (unit 1)
-    (in_bom yes) (on_board yes)
-    (property "Reference" "SW1" (id 0) (at 112.395 46.355 90)
-      (effects (font (size 1.27 1.27)) (justify right))
-    )
-    (property "Value" "SW_SPST" (id 1) (at 109.855 50.165 90)
-      (effects (font (size 1.27 1.27)) (justify right))
-    )
-    (property "Footprint" "" (id 2) (at 120.015 47.625 0)
-      (effects (font (size 1.27 1.27)) hide)
-    )
-    (property "Datasheet" "~" (id 3) (at 120.015 47.625 0)
       (effects (font (size 1.27 1.27)) hide)
     )
@@
     (pin "2")
   )
+  (symbol (lib_id "SamacSys_Parts:PTS526_SK15_SMTR2_LFS") (at 75.565 81.915 0) (unit 1)
+    (in_bom yes) (on_board yes) (fields_autoplaced)
+    (property "Reference" "SW1" (id 0) (at 90.805 73.66 0))
+    (property "Value" "PTS526_SK15_SMTR2_LFS" (id 1) (at 90.805 76.2 0))
+    (property "Footprint" "PTS526SK15SMTR2LFS" (id 2) (at 102.235 79.375 0)
+      (effects (font (size 1.27 1.27)) (justify left) hide)
+    )
+    (property "Datasheet" "https://www.ckswitches.com/media/2780/pts526.pdf" (id 3) (at 102.235 81.915 0)
+      (effects (font (size 1.27 1.27)) (justify left) hide)
+    )
+    (property "Description" "Tact 5.2 x 5.2, 1.5 mm H, 260gf, G leads, No ground pin, metal actuator" (id 4) (at 102.235 84.455 0)
+      (effects (font (size 1.27 1.27)) (justify left) hide)
+    )
+    (property "Height" "1.65" (id 5) (at 102.235 86.995 0)
+      (effects (font (size 1.27 1.27)) (justify left) hide)
+    )
+    (property "Mouser Part Number" "611-PTS526SK15SMR2L" (id 6) (at 102.235 89.535 0)
+      (effects (font (size 1.27 1.27)) (justify left) hide)
+    )
+    (property "Mouser Price/Stock" "https://www.mouser.co.uk/ProductDetail/CK/PTS526-SK15-SMTR2-LFS?qs=UXgszm6BlbF5Ezp94JAQtw%3D%3D" (id 7) (at 102.235 92.075 0)
+      (effects (font (size 1.27 1.27)) (justify left) hide)
+    )
+    (property "Manufacturer_Name" "C & K COMPONENTS" (id 8) (at 102.235 94.615 0)
+      (effects (font (size 1.27 1.27)) (justify left) hide)
+    )
+    (property "Manufacturer_Part_Number" "PTS526 SK15 SMTR2 LFS" (id 9) (at 102.235 97.155 0)
+      (effects (font (size 1.27 1.27)) (justify left) hide)
+    )
+    (pin "1")
+    (pin "2")
+    (pin "3")
+    (pin "4")
+  )
   (symbol (lib_id "SamacSys_Parts:AP2112M-3.3TRG1") (at 93.345 105.41 0) (mirror y) (unit 1)
     (in_bom yes) (on_board yes) (fields_autoplaced)
@@
       (reference "R8") (unit 1) (value "47.5k") (footprint "Resistor_SMD:R_0603_1608Metric_Pad0.98x0.95mm_HandSolder")
     )
-    (path "/1ee31cc3-7d4a-49f7-858c-7c09a0e15095"
-      (reference "SW1") (unit 1) (value "SW_SPST") (footprint "")
+    (path "/fde3844e-a48f-4ec9-a1ca-0d79508f5e3f"
+      (reference "SW1") (unit 1) (value "PTS526_SK15_SMTR2_LFS") (footprint "PTS526SK15SMTR2LFS")
     )
     (path "/740af12e-1e48-4350-b0a0-d48c6545ee1c"

Commit message: f
Parts:
- C1: value 1u -> 100n
- C3: value 0.1u -> 100n
Other:
- moved on the sheet: C4, C5, IC1, J2, J3, J4, Q1A, Q1B, R7, R8
